File: IGBT-Driver-Board/IGBT-Driver-Board.kicad_sch (KiCad schematic)
At the start: 0 parts

Commit message: midnight update 10-4-2026
Other:
- added sheet Driver_Output_DESAT (Driver_Output_DESAT.kicad_sch)
- added sheet IGBT_Stage (IGBT_Zone.kicad_sch)
- added sheet Input_Logic (Input_Logic.kicad_sch)
Changed lines of the file:
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@@
 	(generator_version "10.0")
 	(paper "A4")
+	(sheet
+		(at 151.13 105.41)
+		(size 59.69 22.86)
+		(exclude_from_sim no)
+		(in_bom yes)
+		(on_board yes)
+		(dnp no)
+		(fields_autoplaced yes)
+		(stroke
+			(width 0.1524)
+			(type solid)
+		)
+		(fill
+			(color 0 0 0 0)
+		)
+		(property "Sheetname" "Input_Logic"
+			(at 151.13 104.6984 0)
+			(show_name no)
+			(do_not_autoplace no)
+			(effects
+				(font
+					(size 1.27 1.27)
+				)
+				(justify left bottom)
+			)
+		)
+		(property "Sheetfile" "Input_Logic.kicad_sch"
+			(at 151.13 128.8546 0)
+			(show_name no)
+			(do_not_autoplace no)
+			(effects
+				(font
+					(size 1.27 1.27)
+				)
+				(justify left top)
+			)
+		)
+		(instances
+			(project "IGBT-Driver-Board"
+				(path "/3b56684c-fffd-4181-803c-92224cd33d2a"
+					(page "12")
+				)
+			)
+		)
+	)
+	(sheet
+		(at 33.02 105.41)
+		(size 48.26 17.78)
+		(exclude_from_sim no)
+		(in_bom yes)
+		(on_board yes)
+		(dnp no)
+		(fields_autoplaced yes)
+		(stroke
+			(width 0.1524)
+			(type solid)
+		)
+		(fill
+			(color 0 0 0 0)
+		)
+		(property "Sheetname" "IGBT_Stage"
+			(at 33.02 104.6984 0)
+			(show_name no)
+			(do_not_autoplace no)
+			(effects
+				(font
+					(size 1.27 1.27)
+				)
+				(justify left bottom)
+			)
+		)
+		(property "Sheetfile" "IGBT_Zone.kicad_sch"
+			(at 33.02 123.7746 0)
+			(show_name no)
+			(do_not_autoplace no)
+			(effects
+				(font
+					(size 1.27 1.27)
+				)
+				(justify left top)
+			)
+		)
+		(instances
+			(project "IGBT-Driver-Board"
+				(path "/3b56684c-fffd-4181-803c-92224cd33d2a"
+					(page "2")
+				)
+			)
+		)
+	)
+	(sheet
+		(at 99.06 105.41)
+		(size 30.48 17.78)
+		(exclude_from_sim no)
+		(in_bom yes)
+		(on_board yes)
+		(dnp no)
+		(fields_autoplaced yes)
+		(stroke
+			(width 0.1524)
+			(type solid)
+		)
+		(fill
+			(color 0 0 0 0)
+		)
+		(property "Sheetname" "Driver_Output_DESAT"
+			(at 99.06 104.6984 0)
+			(show_name no)
+			(do_not_autoplace no)
+			(effects
+				(font
+					(size 1.27 1.27)
+				)
+				(justify left bottom)
+			)
+		)
+		(property "Sheetfile" "Driver_Output_DESAT.kicad_sch"
+			(at 99.06 123.7746 0)
+			(show_name no)
+			(do_not_autoplace no)
+			(effects
+				(font
+					(size 1.27 1.27)
+				)
+				(justify left top)
+			)
+		)
+		(instances
+			(project "IGBT-Driver-Board"
+				(path "/3b56684c-fffd-4181-803c-92224cd33d2a"
+					(page "11")
+				)
+			)
+		)
+	)
 	(sheet_instances
 		(path "/"

Commit message: preview 1
Other:
- sheet Input_Logic renamed Gate_Supply
Changed lines of the file:
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@@
 	(paper "A4")
 	(sheet
-		(at 151.13 105.41)
+		(at 175.26 88.9)
 		(size 59.69 22.86)
 		(exclude_from_sim no)
@@
 			(color 0 0 0 0)
 		)
-		(property "Sheetname" "Input_Logic"
-			(at 151.13 104.6984 0)
+		(property "Sheetname" "Gate_Supply"
+			(at 175.26 88.1884 0)
 			(show_name no)
 			(do_not_autoplace no)
@@
 		)
 		(property "Sheetfile" "Input_Logic.kicad_sch"
-			(at 151.13 128.8546 0)
+			(at 175.26 112.3446 0)
 			(show_name no)
 			(do_not_autoplace no)
@@
 	)
 	(sheet
-		(at 33.02 105.41)
+		(at 57.15 88.9)
 		(size 48.26 17.78)
 		(exclude_from_sim no)
@@
 		)
 		(property "Sheetname" "IGBT_Stage"
-			(at 33.02 104.6984 0)
+			(at 57.15 88.1884 0)
 			(show_name no)
 			(do_not_autoplace no)
@@
 		)
 		(property "Sheetfile" "IGBT_Zone.kicad_sch"
-			(at 33.02 123.7746 0)
+			(at 57.15 107.2646 0)
 			(show_name no)
 			(do_not_autoplace no)
@@
 	)
 	(sheet
-		(at 99.06 105.41)
+		(at 123.19 88.9)
 		(size 30.48 17.78)
 		(exclude_from_sim no)
@@
 		)
 		(property "Sheetname" "Driver_Output_DESAT"
-			(at 99.06 104.6984 0)
+			(at 123.19 88.1884 0)
 			(show_name no)
 			(do_not_autoplace no)
@@
 		)
 		(property "Sheetfile" "Driver_Output_DESAT.kicad_sch"
-			(at 99.06 123.7746 0)
+			(at 123.19 107.2646 0)
 			(show_name no)
 			(do_not_autoplace no)
