File: IGBT-Driver-Board/IGBT_Switching_Cell.kicad_sch (KiCad schematic)
At the start: 5 parts, among them Q1 IXEL40N400

Commit message: midnight update 10-5
Parts:
- Q1: footprint Pattarachai's_FootprintLib:IXEL40N400 -> SamacSys_Parts:IXBL60N360
Changed lines of the file:
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@@
 			)
 		)
-		(property "Footprint" "Pattarachai's_FootprintLib:IXEL40N400"
+		(property "Footprint" "SamacSys_Parts:IXBL60N360"
 			(at 157.48 191.44 0)
 			(hide yes)
