File: IGBT-Driver-Board/Driver_Output.kicad_sch (KiCad schematic)
At the start: 18 parts

Commit message: preview 1
Parts:
- renumbered C8 to C23, C9 to C24, C10 to C25, C11 to C26, C12 to C27, D22 to D26, D23 to D27, D24 to D28, D25 to D29, D26 to D30, D27 to D31, D28 to D32, D29 to D33, JP1 to JP2, R26 to R33, R27 to R34, R28 to R35, R29 to R36
Other:
- moved on the sheet: C23, C24, C25, C26, C27, D32, D33, JP2, R36

Commit message: version 1.0.0
Parts:
- C23: value 220p -> 220p, C0G
- C24, C25: value 10u 50V CM -> 10u
- C26, C27: value 100n 50V CM -> 100n
- JP2: value Jumper_2_Open -> DESAT OFF
- R34: value R_PU 4.7k 0.25W -> 4.7k 0.25W
- R35: value R_A 10k 0.25W -> 10k 0.25W
- R36: value R_B 10k 0.25W -> 10k 0.25W
Connections:
- net GATE_BUS: no longer C24.2, C25.1, C26.2, C27.1
- net VCOM: now also C24.2, C25.1, C26.2, C27.1

Commit message: midnight update 10-5
Parts:
- C23: value 220p, C0G -> 220p, C0G 50V; footprint (none) -> SamacSys_Parts:C330C103J5G5TA
- C24, C25: value 10u -> 10u 50V; footprint (none) -> SamacSys_Parts:RDEC71H106K3K1H03B
- C26, C27: value 100n -> 100n 50V; footprint (none) -> SamacSys_Parts:RDER71H104K0M1H03A
- D33: footprint Diode_SMD:D_01005_0402Metric -> Diode_THT:D_DO-41_SOD81_P10.16mm_Horizontal
- JP2: footprint TestPoint:TestPoint_2Pads_Pitch2.54mm_Drill0.8mm -> Connector_PinHeader_2.54mm:PinHeader_1x02_P2.54mm_Vertical
Changed lines of the file:
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@@
 		(in_pos_files yes)
 		(dnp no)
-		(fields_autoplaced yes)
 		(property "Reference" "C24"
 			(at 203.2 97.7899 0)
@@
 			)
 		)
-		(property "Value" "10u"
+		(property "Value" "10u 50V"
 			(at 203.2 100.3299 0)
 			(show_name no)
@@
 			)
 		)
-		(property "Footprint" ""
+		(property "Footprint" "SamacSys_Parts:RDEC71H106K3K1H03B"
 			(at 200.3552 102.87 0)
 			(hide yes)
@@
 			)
 		)
-		(property "Description" "Unpolarized capacitor"
-			(at 199.39 99.06 0)
-			(hide yes)
+		(property "Description" ""
+			(at 209.55 99.06 0)
 			(show_name no)
 			(do_not_autoplace no)
@@
 			)
 		)
-		(property "Value" "220p, C0G"
+		(property "Value" "220p, C0G 50V"
 			(at 167.64 97.7899 0)
 			(show_name no)
@@
 			)
 		)
-		(property "Footprint" ""
+		(property "Footprint" "SamacSys_Parts:C330C103J5G5TA"
 			(at 164.7952 100.33 0)
 			(hide yes)
@@
 		(in_pos_files yes)
 		(dnp no)
-		(fields_autoplaced yes)
 		(property "Reference" "C26"
 			(at 223.52 97.7899 0)
@@
 			)
 		)
-		(property "Value" "100n"
+		(property "Value" "100n 50V"
 			(at 223.52 100.3299 0)
 			(show_name no)
@@
 			)
 		)
-		(property "Footprint" ""
+		(property "Footprint" "SamacSys_Parts:RDER71H104K0M1H03A"
 			(at 220.6752 102.87 0)
 			(hide yes)
@@
 			)
 		)
-		(property "Description" "Unpolarized capacitor"
-			(at 219.71 99.06 0)
-			(hide yes)
+		(property "Description" ""
+			(at 229.87 99.06 0)
 			(show_name no)
 			(do_not_autoplace no)
@@
 			)
 		)
-		(property "Footprint" "TestPoint:TestPoint_2Pads_Pitch2.54mm_Drill0.8mm"
+		(property "Footprint" "Connector_PinHeader_2.54mm:PinHeader_1x02_P2.54mm_Vertical"
 			(at 92.71 96.52 0)
 			(hide yes)
@@
 		(in_pos_files yes)
 		(dnp no)
-		(fields_autoplaced yes)
 		(property "Reference" "C27"
 			(at 223.52 107.9499 0)
@@
 			)
 		)
-		(property "Value" "100n"
+		(property "Value" "100n 50V"
 			(at 223.52 110.4899 0)
 			(show_name no)
@@
 			)
 		)
-		(property "Footprint" ""
+		(property "Footprint" "SamacSys_Parts:RDER71H104K0M1H03A"
 			(at 220.6752 113.03 0)
 			(hide yes)
@@
 			)
 		)
-		(property "Description" "Unpolarized capacitor"
-			(at 219.71 109.22 0)
-			(hide yes)
+		(property "Description" ""
+			(at 229.87 109.22 0)
 			(show_name no)
 			(do_not_autoplace no)
@@
 		(in_pos_files yes)
 		(dnp no)
-		(fields_autoplaced yes)
 		(property "Reference" "C25"
 			(at 203.2 107.9499 0)
@@
 			)
 		)
-		(property "Value" "10u"
+		(property "Value" "10u 50V"
 			(at 203.2 110.4899 0)
 			(show_name no)
@@
 			)
 		)
-		(property "Footprint" ""
+		(property "Footprint" "SamacSys_Parts:RDEC71H106K3K1H03B"
 			(at 200.3552 113.03 0)
 			(hide yes)
@@
 			)
 		)
-		(property "Description" "Unpolarized capacitor"
-			(at 199.39 109.22 0)
-			(hide yes)
+		(property "Description" ""
+			(at 209.55 109.22 0)
 			(show_name no)
 			(do_not_autoplace no)
@@
 			)
 		)
-		(property "Footprint" "Diode_SMD:D_01005_0402Metric"
+		(property "Footprint" "Diode_THT:D_DO-41_SOD81_P10.16mm_Horizontal"
 			(at 125.095 96.52 0)
 			(hide yes)

Commit message: version 2.0.0
Changed lines of the file:
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@@
 			)
 		)
-		(property "Description" ""
+		(property "Description" "Unpolarized capacitor"
 			(at 209.55 99.06 0)
 			(show_name no)
@@
 			)
 		)
-		(property "Description" ""
+		(property "Description" "Unpolarized capacitor"
 			(at 229.87 99.06 0)
 			(show_name no)
@@
 			)
 		)
-		(property "Description" ""
+		(property "Description" "Unpolarized capacitor"
 			(at 229.87 109.22 0)
 			(show_name no)
@@
 			)
 		)
-		(property "Description" ""
+		(property "Description" "Unpolarized capacitor"
 			(at 209.55 109.22 0)
 			(show_name no)
