File: IGBT-Driver-Board/Driver_Output_DESAT.kicad_sch (KiCad schematic)
At the start: 29 parts, among them IC1 CD74HC14E, J1 HFBR-2521Z, J2 HFBR-2521Z, U1 UCC21750QDWRQ1

Commit message: preview 1
Parts:
- added C3: 10n, symbol Device:C
- added C7: 22u, symbol Device:C
- added C8: 100n, symbol Device:C
- added D21: Green, LED_THT:LED_D5.0mm_Clear, symbol Device:LED
- added F1: PTC 0.65A, Connector_Wire:SolderWire-1.5sqmm_1x02_P6mm_D1.7mm_OD3mm, symbol Device:Polyfuse
- added IC1: CD74HC221E, SamacSys_Parts:DIP794W53P254L1930H508Q16N, symbol SamacSys:CD74HC221E
- added J1: TEST, Connector_PinHeader_2.54mm:PinHeader_1x03_P2.54mm_Vertical, symbol Connector:Conn_01x03_Pin
- added J4: Input Power, TerminalBlock_Phoenix:TerminalBlock_Phoenix_MKDS-1,5-2_1x02_P5.00mm_Horizontal, symbol Connector:Screw_Terminal_01x02
- added R21: 4.7k 0.25W, Resistor_THT:R_Axial_DIN0207_L6.3mm_D2.5mm_P10.16mm_Horizontal, symbol Device:R_US
- added R22: 3296W-1-104, SamacSys_Parts:3296W1503LF, symbol SamacSys:3296W-1-104
- added R26: 1k 0.25W, Resistor_THT:R_Axial_DIN0207_L6.3mm_D2.5mm_P10.16mm_Horizontal, symbol Device:R_US
- renumbered C5 to C10, C6 to C11, C7 to C12, C13 to C4, C3 to C5, C14 to C6, C4 to C9, D30 to D19, D19 to D20, D21 to D22, D20 to D23, IC1 to IC2, J1 to J2, J2 to J3, R30 to R17, R17 to R18, R31 to R19, R18 to R20, R32 to R23, R19 to R24, R24 to R27, R22 to R28, R21 to R29, R20 to R30, R23 to R31
Connections:
- net +5V: now also C7.1, C8.1, F1.2, IC1.16 (VCC), R22.1 (CCW), R26.2
- net EN: now also IC1.3 (~{1R})
- net EN_RX_N: now also J1.2 (Pin_2)
- net FIRE_P: now also IC1.2 (1B)
- net FIRE_RX_N: now also J1.1 (Pin_1)
- net GNDREF: now also IC2.11 (5A), IC2.13 (6A), C7.2, C8.2, D21.1 (K), IC1.1 (~{1A}), IC1.10 (2B), IC1.11 (~{2R}), IC1.8 (GND), IC1.9 (~{2A}), J1.3 (Pin_3), J4.2 (Pin_2)
- net at R29.2: now also IC1.13 (1Q)
- new net: F1.1, J4.1 (Pin_1)
- new net: C3.1, IC1.14 (1CX)
- new net: C3.2, IC1.15 (1CXRX), R21.2
- new net: D21.2 (A), R26.1
- new net: R21.1, R22.2 (WIPER), R22.3 (CW)
- no-connect marks 3 -> 10
Other:
- moved on the sheet: C1, C2, C4, C5, C6, D19, D20, D22, D23, IC2, J2, J3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

Commit message: version 1.0.0
Parts:
- C10: value 100n, U1 -> 100n
- C11: value 1u, U3 -> 1u
- C12: value 100n, U3 -> 100n
- C3: value 10n -> 10n, C0G
- C4: value 1n -> 1n, C0G
- C6: value 470p -> 470p, C0G
- C9: value 100n, U2 -> 100n
- R21: value 4.7k 0.25W -> 2.7k 0.25W
- R22: value 3296W-1-104 -> 3296W-1-102
Changed lines of the file:
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@@
 			(font
 				(size 1.27 1.27)
+				(thickness 0.1588)
 			)
 			(justify right bottom)
@@
 			)
 		)
-		(property "Value" "1n"
+		(property "Value" "1n, C0G"
 			(at 97.79 101.6 0)
 			(show_name no)
@@
 			)
 		)
-		(property "Value" "3296W-1-104"
+		(property "Value" "3296W-1-102"
 			(at 110.49 33.02 0)
 			(show_name no)
@@
 		(dnp no)
 		(property "Reference" "C6"
-			(at 101.6 88.9 90)
+			(at 102.87 88.9 90)
 			(show_name no)
 			(do_not_autoplace no)
@@
 			)
 		)
-		(property "Value" "470p"
-			(at 101.6 91.44 90)
+		(property "Value" "470p, C0G"
+			(at 99.06 91.44 90)
 			(show_name no)
 			(do_not_autoplace no)
@@
 		(dnp no)
 		(property "Reference" "C3"
-			(at 85.725 36.195 90)
+			(at 85.09 43.18 90)
 			(show_name no)
 			(do_not_autoplace no)
@@
 			)
 		)
-		(property "Value" "10n"
-			(at 85.725 33.655 90)
+		(property "Value" "10n, C0G"
+			(at 88.9 45.72 90)
 			(show_name no)
 			(do_not_autoplace no)
@@
 			)
 		)
-		(property "Value" "100n, U2"
+		(property "Value" "100n"
 			(at 223.52 153.67 0)
 			(show_name no)
@@
 			)
 		)
-		(property "Description" "Unpolarized capacitor"
-			(at 220.98 152.4 0)
-			(hide yes)
+		(property "Description" "U2"
+			(at 223.52 156.21 0)
 			(show_name no)
 			(do_not_autoplace no)
@@
 			)
 		)
-		(property "Value" "1u, U3"
+		(property "Value" "1u"
 			(at 254 153.67 0)
 			(show_name no)
@@
 			)
 		)
-		(property "Description" "Unpolarized capacitor"
-			(at 251.46 152.4 0)
-			(hide yes)
+		(property "Description" "U3"
+			(at 254 156.21 0)
 			(show_name no)
 			(do_not_autoplace no)
@@
 			)
 		)
-		(property "Value" "4.7k 0.25W"
+		(property "Value" "2.7k 0.25W"
 			(at 97.79 35.56 90)
 			(show_name no)
@@
 			)
 		)
-		(property "Value" "100n, U1"
+		(property "Value" "100n"
 			(at 238.76 153.67 0)
 			(show_name no)
@@
 			)
 		)
-		(property "Description" "Unpolarized capacitor"
-			(at 236.22 152.4 0)
-			(hide yes)
+		(property "Description" "U1"
+			(at 238.76 156.21 0)
 			(show_name no)
 			(do_not_autoplace no)
@@
 			)
 		)
-		(property "Value" "100n, U3"
+		(property "Value" "100n"
 			(at 266.7 153.67 0)
 			(show_name no)
@@
 			)
 		)
-		(property "Description" "Unpolarized capacitor"
-			(at 264.16 152.4 0)
-			(hide yes)
+		(property "Description" "U3"
+			(at 266.7 156.21 0)
 			(show_name no)
 			(do_not_autoplace no)

Commit message: midnight update 10-5
Parts:
- removed C7: 22u, symbol Device:C
- removed F1: PTC 0.65A, Connector_Wire:SolderWire-1.5sqmm_1x02_P6mm_D1.7mm_OD3mm, symbol Device:Polyfuse
- added C7: 22u, Capacitor_THT:CP_Radial_D5.0mm_P2.00mm, symbol Device:C_Polarized
- added F2: RXEF065, SamacSys_Parts:RXEF065, symbol SamacSys:RXEF065
- C1, C10, C12, C2, C5, C8, C9: footprint (none) -> SamacSys_Parts:RDER71H104K0M1H03A
- C11: footprint (none) -> Pattarachai's_FootprintLib:K105M20X7RF5UH5_VIS
- C3, C4, C6: footprint (none) -> SamacSys_Parts:C330C103J5G5TA
Connections:
- net +5V: now also C7.1, F2.2
- net GNDREF: now also C7.2
- net at J4.1 (Pin_1): now also F2.1
Other:
- moved on the sheet: C8, D21, R26

Commit message: version 2.0.0
Parts:
- F2: footprint SamacSys_Parts:RXEF065 -> RXEF065
Changed lines of the file:
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@@
 			)
 		)
-		(property "Description" "IC1"
+		(property "Description" "Unpolarized capacitor"
 			(at 223.52 156.21 0)
 			(show_name no)
@@
 			)
 		)
-		(property "Description" "U1"
-			(at 254 156.21 0)
+		(property "Description" "Unpolarized capacitor"
+			(at 252.73 160.02 0)
 			(show_name no)
 			(do_not_autoplace no)
@@
 			)
 		)
-		(property "Footprint" "SamacSys_Parts:RXEF065"
+		(property "Footprint" "RXEF065"
 			(at 95.25 276.53 0)
 			(hide yes)
@@
 	)
 	(symbol
-		(lib_name "HFBR-2521Z_1")
 		(lib_id "Pattarachai's_Lib:HFBR-2521Z")
 		(at 64.77 130.81 0)
@@
 			)
 		)
-		(property "Description" "IC2"
-			(at 238.76 156.21 0)
+		(property "Description" "Unpolarized capacitor"
+			(at 238.76 161.29 0)
 			(show_name no)
 			(do_not_autoplace no)
@@
 			)
 		)
-		(property "Description" "U1"
-			(at 266.7 156.21 0)
+		(property "Description" "Unpolarized capacitor"
+			(at 265.43 160.02 0)
 			(show_name no)
 			(do_not_autoplace no)
