File: IGBT-Driver-Board/IGBT-Driver-Board.kicad_pcb (KiCad board)
At the start: 2 copper layers, 276.1 x 165.3 mm, 117 parts, among them IC1 CD74HC221E, IC2 CD74HC14E, J1 TEST, J2 HFBR-2521Z, J3 HFBR-2521Z, J4 Input Power, J5 74655095R, J6 74655095R, Q1 IXEL40N400, Q2 IXEL40N400, Q3 IXEL40N400, Q4 IXEL40N400, Q5 IXEL40N400, Q6 IXEL40N400, Q7 IXEL40N400, Q8 IXEL40N400, U1 UCC21750QDWRQ1, U2 MGJ2D051515SC

Commit message: version 2.0.0
Parts:
- added NT1: NetTie_2, Pattarachai's_FootprintLib:NetTie-2_SMD_Pad6.0mm, B.Cu at (92.0, 102.9)
- added U3: ~, Pattarachai's_FootprintLib:Heatsink_150x20x6mm, F.Cu at (91.3, 107.4)
- added U4: ~, Pattarachai's_FootprintLib:Heatsink_150x20x6mm_flip, F.Cu at (241.3, 98.3)
- moved D1 193.9 mm to (264.7, 70.4), turned to 180 degrees
- moved D2 190.9 mm to (264.7, 64.1), turned to 180 degrees
- moved D26 165.1 mm to (244.0, 44.5), turned to 180 degrees
- moved D27 149.3 mm to (228.7, 44.5), turned to 180 degrees
- moved D28 133.6 mm to (213.5, 44.5), turned to 180 degrees
- moved R17 131.8 mm to (75.9, 133.9), turned to 180 degrees
- moved R24 129.5 mm to (89.9, 147.3)
- moved J2 126.7 mm to (72.6, 139.7)
- moved J3 122.0 mm to (54.5, 139.7)
- moved R19 121.0 mm to (75.9, 129.8), turned to 180 degrees
- moved R18 120.4 mm to (55.8, 134.1), turned to 180 degrees
- moved D20 119.5 mm to (90.2, 154.4), turned to 90 degrees
- moved R25 119.3 mm to (77.2, 147.3)
- moved D31 117.1 mm to (198.2, 44.5), turned to 180 degrees
- moved R31 112.0 mm to (100.1, 143.6), turned to 180 degrees
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Routing:
- net GATE_BUS: track 294.3 -> 654.0 mm
- net VDD: track 0.00 -> 132.4 mm
- net /Driver_Output_DESAT/Driver_Output/DESAT: track 0.00 -> 121.7 mm
- net EN: track 0.00 -> 101.5 mm
- net VEE: track 0.00 -> 92.8 mm
- net Net-(D22-K): track 0.00 -> 66.0 mm
- net FIRE_RX_N: track 0.00 -> 58.0 mm
- net /Driver_Output_DESAT/FIRE_P: track 0.00 -> 56.3 mm
- net Net-(IC2-2A): track 0.00 -> 52.7 mm
- net RDY: track 0.00 -> 48.5 mm
- net VCOM: track 0.00 -> 40.8 mm
- net EN_RX_N: track 0.00 -> 40.0 mm
- net Net-(D19-A): track 0.00 -> 38.7 mm
- net Net-(R22-CW): track 0.00 -> 28.4 mm
- net Net-(D23-K): track 0.00 -> 28.2 mm
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- added copper zone on F.Cu, net +5V
- added copper zone on F.Cu, net E_BUS
- added copper zone on B.Cu, net GNDREF
- added copper zone on B.Cu, net VCOM
- added copper zone on F.Cu, net VCOM
Other:
- board size 276.1 x 165.3 mm -> 245 x 127 mm
- board text added: "+HV"
- board text added: "5V GND -15 0 15"
- board text added: "5Vin GND"
- board text added: "GND"
- board text added: "MPC"
- board text added: "Pattarachai Bor-in"
- board text added: "U3"
