File: IGBT-Driver-Board/IGBT_Zone.kicad_sch (KiCad schematic)
At the start: 2 parts

Commit message: version 1.0.0
Parts:
- added J5, J6: 74655095R, SamacSys_Parts:74655095R, symbol SamacSys:74655095R
- added NT1: NetTie_2, symbol Device:NetTie_2
Connections:
- net C_BUS: now also J5.1, J5.2, J5.3, J5.4, J5.5, J5.6, J5.7, J5.8
- net E_BUS: now also J6.1, J6.2, J6.3, J6.4, J6.5, J6.6, J6.7, J6.8, NT1.2
- new net VCOM: NT1.1

Commit message: midnight update 10-5
Parts:
- D1, D2: footprint Diode_THT:D_DO-41_SOD81_P10.16mm_Horizontal -> Pattarachai's_FootprintLib:D_DO-41_P20.32mm_HV_Horizontal
Changed lines of the file:
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@@
 			)
 		)
-		(property "Footprint" "Diode_THT:D_DO-41_SOD81_P10.16mm_Horizontal"
+		(property "Footprint" "Pattarachai's_FootprintLib:D_DO-41_P20.32mm_HV_Horizontal"
 			(at 166.37 48.26 0)
 			(hide yes)
@@
 			)
 		)
-		(property "Footprint" "Diode_THT:D_DO-41_SOD81_P10.16mm_Horizontal"
+		(property "Footprint" "Pattarachai's_FootprintLib:D_DO-41_P20.32mm_HV_Horizontal"
 			(at 180.34 48.26 0)
 			(hide yes)

Commit message: version 2.0.0
Parts:
- added U3: (no value), Pattarachai's_FootprintLib:Heatsink_150x20x6mm, symbol Pattarachai's_Lib:Heatsink_150x20x6mm
- added U4: (no value), Pattarachai's_FootprintLib:Heatsink_150x20x6mm_flip, symbol Pattarachai's_Lib:Heatsink_150x20x6mm_flip
- NT1: footprint (none) -> Pattarachai's_FootprintLib:NetTie-2_SMD_Pad6.0mm
Connections:
- net E_BUS: now also U3.1 (H1), U3.2 (H2), U4.1 (H1), U4.2 (H2)
