File: IGBT-Driver-Board/Input_Logic.kicad_sch (KiCad schematic)
At the start: 0 parts

Commit message: preview 1
Parts:
- added C13: 4.7u, symbol Device:C
- added C14: 1u, 50V, symbol Device:C
- added C15, C16, C17, C18: 10u, 50V, symbol Device:C
- added C19, C20: 47µF, 50V, symbol Device:C_Polarized
- added C21, C22: 100n, 50V, symbol Device:C
- added D24, D25: 1N4733A 5.1V, Diode_THT:D_DO-41_SOD81_P7.62mm_Horizontal, symbol Device:D_Zener
- added JP1: MODE, TestPoint:TestPoint_2Pads_Pitch2.54mm_Drill0.8mm, symbol Jumper:Jumper_2_Open
- added R32: 2.2k 2W, Resistor_THT:R_Axial_DIN0516_L15.5mm_D5.0mm_P20.32mm_Horizontal, symbol Device:R_US
- added U2: MGJ2D051515SC, Pattarachai's_FootprintLib:MGJ2_MUR, symbol Pattarachai's_Lib:MGJ2D051515SC
Connections:
- new net: C14.1, D24.1 (K), JP1.2 (B), U2.7 (+Vout)
- new net +5V: C13.1, U2.1 (+Vin)
- new net COM: C15.2, C16.1, C17.2, C18.1, C19.2, C20.1, C21.2, C22.1, D25.1 (K), R32.1
- new net GNDREF: C13.2, U2.2 (-Vin)
- new net VDD: C15.1, C17.1, C19.1, C21.1, D24.2 (A), JP1.1 (A), R32.2
- new net VEE: C14.2, C16.2, C18.2, C20.2, C22.2, D25.2 (A), U2.5 (-Vout)
- no-connect marks 0 -> 1

Commit message: version 1.0.0
Parts:
- C14: value 1u, 50V -> 1u
- C15, C16, C17, C18: value 10u, 50V -> 10u
- C19, C20: value 47µF, 50V -> 47u
- C21, C22: value 100n, 50V -> 100n
Connections:
- net COM renamed VCOM
Changed lines of the file:
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@@
+	)
+	(junction
+		(at 115.57 114.3)
+		(diameter 0)
+		(color 0 0 0 0)
 	)
 	(junction
@@
 	)
 	(junction
-		(at 115.57 93.98)
-		(diameter 0)
-		(color 0 0 0 0)
-	)
-	(junction
 		(at 55.88 97.79)
 		(diameter 0)
@@
 	)
 	(junction
+		(at 115.57 93.98)
+		(diameter 0)
+		(color 0 0 0 0)
+	)
+	(junction
 		(at 187.96 80.01)
 		(diameter 0)
@@
 	)
 	(junction
-		(at 115.57 114.3)
-		(diameter 0)
-		(color 0 0 0 0)
-	)
-	(junction
 		(at 201.93 80.01)
 		(diameter 0)
@@
 	(wire
 		(pts
-			(xy 101.6 114.3) (xy 115.57 114.3)
+			(xy 102.87 114.3) (xy 115.57 114.3)
 		)
 		(stroke
@@
 	(wire
 		(pts
+			(xy 102.87 106.68) (xy 101.6 106.68)
+		)
+		(stroke
+			(width 0)
+			(type default)
+		)
+	)
+	(wire
+		(pts
 			(xy 175.26 96.52) (xy 175.26 101.6)
 		)
@@
 	(wire
 		(pts
-			(xy 101.6 93.98) (xy 115.57 93.98)
+			(xy 102.87 93.98) (xy 115.57 93.98)
 		)
 		(stroke
@@
 	(wire
 		(pts
-			(xy 101.6 106.68) (xy 101.6 114.3)
+			(xy 102.87 106.68) (xy 102.87 114.3)
 		)
 		(stroke
@@
 	(wire
 		(pts
+			(xy 102.87 101.6) (xy 101.6 101.6)
+		)
+		(stroke
+			(width 0)
+			(type default)
+		)
+	)
+	(wire
+		(pts
 			(xy 163.83 114.3) (xy 175.26 114.3)
 		)
@@
 	(wire
 		(pts
+			(xy 279.4 157.48) (xy 279.4 154.94)
+		)
+		(stroke
+			(width 0)
+			(type default)
+		)
+	)
+	(wire
+		(pts
 			(xy 175.26 96.52) (xy 187.96 96.52)
 		)
@@
 	(wire
 		(pts
-			(xy 101.6 101.6) (xy 101.6 93.98)
+			(xy 102.87 101.6) (xy 102.87 93.98)
 		)
 		(stroke
@@
 		)
 	)
-	(global_label "COM"
+	(global_label "VDD"
 		(shape input)
-		(at 234.95 96.52 0)
+		(at 279.4 157.48 270)
 		(fields_autoplaced yes)
 		(effects
@@
 				(size 1.27 1.27)
 			)
-			(justify left)
+			(justify right)
 		)
 		(property "Intersheetrefs" "${INTERSHEET_REFS}"
-			(at 241.9871 96.52 0)
-			(hide yes)
-			(show_name no)
-			(do_not_autoplace no)
-			(effects
-				(font
-					(size 1.27 1.27)
-				)
-				(justify left)
+			(at 279.4 164.0938 90)
+			(hide yes)
+			(show_name no)
+			(do_not_autoplace no)
+			(effects
+				(font
+					(size 1.27 1.27)
+				)
+				(justify right)
 			)
 		)
@@
 			)
 		)
-		(property "Value" "100n, 50V"
+		(property "Value" "100n"
 			(at 203.2 101.6 0)
 			(show_name no)
@@
 			)
 		)
-		(property "Value" "47µF, 50V"
+		(property "Value" "47u"
 			(at 189.23 102.87 0)
 			(show_name no)
@@
 	)
 	(symbol
+		(lib_id "power:VCOM")
+		(at 234.95 96.52 270)
+		(unit 1)
+		(body_style 1)
+		(exclude_from_sim no)
+		(in_bom yes)
+		(on_board yes)
+		(in_pos_files yes)
+		(dnp no)
+		(fields_autoplaced yes)
+		(property "Reference" "#PWR041"
+			(at 231.14 96.52 0)
+			(hide yes)
+			(show_name no)
+			(do_not_autoplace no)
+			(effects
+				(font
+					(size 1.27 1.27)
+				)
+			)
+		)
+		(property "Value" "VCOM"
+			(at 238.76 96.5199 90)
+			(show_name no)
+			(do_not_autoplace no)
+			(effects
+				(font
+					(size 1.27 1.27)
+				)
+				(justify left)
+			)
+		)
+		(property "Footprint" ""
+			(at 234.95 96.52 0)
+			(hide yes)
+			(show_name no)
+			(do_not_autoplace no)
+			(effects
+				(font
+					(size 1.27 1.27)
+				)
+			)
+		)
+		(property "Datasheet" ""
+			(at 234.95 96.52 0)
+			(hide yes)
+			(show_name no)
+			(do_not_autoplace no)
+			(effects
+				(font
+					(size 1.27 1.27)
+				)
+			)
+		)
+		(property "Description" "Power symbol creates a global label with name \"VCOM\""
+			(at 234.95 96.52 0)
+			(hide yes)
+			(show_name no)
+			(do_not_autoplace no)
+			(effects
+				(font
+					(size 1.27 1.27)
+				)
+			)
+		)
+		(pin "1"
+		)
+		(instances
+			(project "IGBT-Driver-Board"
+				(path "/3b56684c-fffd-4181-803c-92224cd33d2a/96774f39-b093-412e-8f8f-b317b1308084"
+					(reference "#PWR041")
+					(unit 1)
+				)
+			)
+		)
+	)
+	(symbol
 		(lib_id "Device:C_Polarized")
 		(at 187.96 87.63 0)
@@
 			)
 		)
-		(property "Value" "47µF, 50V"
+		(property "Value" "47u"
 			(at 189.23 85.09 0)
 			(show_name no)
@@
 			)
 		)
-		(property "Value" "1u, 50V"
+		(property "Value" "1u"
 			(at 119.38 105.41 0)
 			(show_name no)
@@
 			)
 		)
-		(property "Value" "10u, 50V"
+		(property "Value" "10u"
 			(at 176.53 85.09 0)
 			(show_name no)
@@
 			)
 		)
-		(property "Value" "100n, 50V"
+		(property "Value" "100n"
 			(at 203.2 85.09 0)
 			(show_name no)
@@
 	)
 	(symbol
+		(lib_id "power:PWR_FLAG")
+		(at 279.4 154.94 0)
+		(unit 1)
+		(body_style 1)
+		(exclude_from_sim no)
+		(in_bom yes)
+		(on_board yes)
+		(in_pos_files yes)
+		(dnp no)
+		(fields_autoplaced yes)
+		(property "Reference" "#FLG03"
+			(at 279.4 153.035 0)
+			(hide yes)
+			(show_name no)
+			(do_not_autoplace no)
+			(effects
+				(font
+					(size 1.27 1.27)
+				)
+			)
+		)
+		(property "Value" "PWR_FLAG"
+			(at 279.4 149.86 0)
+			(hide yes)
+			(show_name no)
+			(do_not_autoplace no)
+			(effects
+				(font
+					(size 1.27 1.27)
+				)
+			)
+		)
+		(property "Footprint" ""
+			(at 279.4 154.94 0)
+			(hide yes)
+			(show_name no)
+			(do_not_autoplace no)
+			(effects
+				(font
+					(size 1.27 1.27)
+				)
+			)
+		)
+		(property "Datasheet" ""
+			(at 279.4 154.94 0)
+			(hide yes)
+			(show_name no)
+			(do_not_autoplace no)
+			(effects
+				(font
+					(size 1.27 1.27)
+				)
+			)
+		)
+		(property "Description" "Special symbol for telling ERC where power comes from"
+			(at 279.4 154.94 0)
+			(hide yes)
+			(show_name no)
+			(do_not_autoplace no)
+			(effects
+				(font
+					(size 1.27 1.27)
+				)
+			)
+		)
+		(pin "1"
+		)
+		(instances
+			(project "IGBT-Driver-Board"
+				(path "/3b56684c-fffd-4181-803c-92224cd33d2a/96774f39-b093-412e-8f8f-b317b1308084"
+					(reference "#FLG03")
+					(unit 1)
+				)
+			)
+		)
+	)
+	(symbol
 		(lib_id "Device:D_Zener")
 		(at 133.35 86.36 90)
@@
 			)
 		)
-		(property "Value" "10u, 50V"
+		(property "Value" "10u"
 			(at 165.1 85.09 0)
 			(show_name no)
@@
 			)
 		)
-		(property "Value" "10u, 50V"
+		(property "Value" "10u"
 			(at 165.1 101.6 0)
 			(show_name no)
@@
 			)
 		)
-		(property "Value" "10u, 50V"
+		(property "Value" "10u"
 			(at 176.53 101.6 0)
 			(show_name no)

Commit message: midnight update 10-5
Parts:
- C13: footprint (none) -> SamacSys_Parts:RDEC71H475K2M1H03A
- C14: value 1u -> 1u 50V; footprint (none) -> Pattarachai's_FootprintLib:K105M20X7RF5UH5_VIS
- C15, C16, C17, C18: value 10u -> 10u 50V; footprint (none) -> SamacSys_Parts:RDEC71H106K3K1H03B
- C19, C20: value 47u -> 47u 50V; footprint (none) -> Capacitor_THT:CP_Radial_D6.3mm_P2.50mm
- C21, C22: value 100n -> 100n 50V; footprint (none) -> SamacSys_Parts:RDER71H104K0M1H03A
- JP1: footprint TestPoint:TestPoint_2Pads_Pitch2.54mm_Drill0.8mm -> Connector_PinHeader_2.54mm:PinHeader_1x02_P2.54mm_Vertical
Changed lines of the file:
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@@
 			)
 		)
-		(property "Value" "100n"
+		(property "Value" "100n 50V"
 			(at 203.2 101.6 0)
 			(show_name no)
@@
 			)
 		)
-		(property "Footprint" ""
+		(property "Footprint" "SamacSys_Parts:RDER71H104K0M1H03A"
 			(at 202.8952 109.22 0)
 			(hide yes)
@@
 			)
 		)
-		(property "Description" "Unpolarized capacitor"
-			(at 201.93 105.41 0)
-			(hide yes)
+		(property "Description" ""
+			(at 204.47 109.22 0)
 			(show_name no)
 			(do_not_autoplace no)
@@
 			)
 		)
-		(property "Value" "47u"
+		(property "Value" "47u 50V"
 			(at 189.23 102.87 0)
 			(show_name no)
@@
 			)
 		)
-		(property "Footprint" ""
+		(property "Footprint" "Capacitor_THT:CP_Radial_D6.3mm_P2.50mm"
 			(at 188.9252 109.22 0)
 			(hide yes)
@@
 			)
 		)
-		(property "Description" "Polarized capacitor"
-			(at 187.96 105.41 0)
-			(hide yes)
+		(property "Description" ""
+			(at 190.5 109.22 0)
 			(show_name no)
 			(do_not_autoplace no)
@@
 			)
 		)
-		(property "Value" "47u"
+		(property "Value" "47u 50V"
 			(at 189.23 85.09 0)
 			(show_name no)
@@
 			)
 		)
-		(property "Footprint" ""
+		(property "Footprint" "Capacitor_THT:CP_Radial_D6.3mm_P2.50mm"
 			(at 188.9252 91.44 0)
 			(hide yes)
@@
 			)
 		)
-		(property "Description" "Polarized capacitor"
-			(at 187.96 87.63 0)
-			(hide yes)
+		(property "Description" ""
+			(at 190.5 91.44 0)
 			(show_name no)
 			(do_not_autoplace no)
@@
 			)
 		)
-		(property "Value" "1u"
+		(property "Value" "1u 50V"
 			(at 119.38 105.41 0)
 			(show_name no)
@@
 			)
 		)
-		(property "Footprint" ""
+		(property "Footprint" "Pattarachai's_FootprintLib:K105M20X7RF5UH5_VIS"
 			(at 116.5352 107.95 0)
 			(hide yes)
@@
 			)
 		)
-		(property "Description" "Unpolarized capacitor"
-			(at 115.57 104.14 0)
-			(hide yes)
+		(property "Description" ""
+			(at 118.11 107.95 0)
 			(show_name no)
 			(do_not_autoplace no)
@@
 			)
 		)
-		(property "Value" "10u"
+		(property "Value" "10u 50V"
 			(at 176.53 85.09 0)
 			(show_name no)
@@
 			)
 		)
-		(property "Footprint" ""
+		(property "Footprint" "SamacSys_Parts:RDEC71H106K3K1H03B"
 			(at 176.2252 91.44 0)
 			(hide yes)
@@
 			)
 		)
-		(property "Description" "Unpolarized capacitor"
-			(at 175.26 87.63 0)
-			(hide yes)
+		(property "Description" ""
+			(at 177.8 91.44 0)
 			(show_name no)
 			(do_not_autoplace no)
@@
 			)
 		)
-		(property "Value" "100n"
+		(property "Value" "100n 50V"
 			(at 203.2 85.09 0)
 			(show_name no)
@@
 			)
 		)
-		(property "Footprint" ""
+		(property "Footprint" "SamacSys_Parts:RDER71H104K0M1H03A"
 			(at 202.8952 91.44 0)
 			(hide yes)
@@
 			)
 		)
-		(property "Description" "Unpolarized capacitor"
-			(at 201.93 87.63 0)
-			(hide yes)
+		(property "Description" ""
+			(at 204.47 91.44 0)
 			(show_name no)
 			(do_not_autoplace no)
@@
 			)
 		)
-		(property "Footprint" ""
+		(property "Footprint" "SamacSys_Parts:RDEC71H475K2M1H03A"
 			(at 56.8452 106.68 0)
 			(hide yes)
@@
 			)
 		)
-		(property "Value" "10u"
+		(property "Value" "10u 50V"
 			(at 165.1 85.09 0)
 			(show_name no)
@@
 			)
 		)
-		(property "Footprint" ""
+		(property "Footprint" "SamacSys_Parts:RDEC71H106K3K1H03B"
 			(at 164.7952 91.44 0)
 			(hide yes)
@@
 			)
 		)
-		(property "Description" "Unpolarized capacitor"
-			(at 163.83 87.63 0)
-			(hide yes)
+		(property "Description" ""
+			(at 166.37 91.44 0)
 			(show_name no)
 			(do_not_autoplace no)
@@
 			)
 		)
-		(property "Footprint" "TestPoint:TestPoint_2Pads_Pitch2.54mm_Drill0.8mm"
+		(property "Footprint" "Connector_PinHeader_2.54mm:PinHeader_1x02_P2.54mm_Vertical"
 			(at 143.51 87.63 0)
 			(hide yes)
@@
 			)
 		)
-		(property "Value" "10u"
+		(property "Value" "10u 50V"
 			(at 165.1 101.6 0)
 			(show_name no)
@@
 			)
 		)
-		(property "Footprint" ""
+		(property "Footprint" "SamacSys_Parts:RDEC71H106K3K1H03B"
 			(at 164.7952 109.22 0)
 			(hide yes)
@@
 			)
 		)
-		(property "Description" "Unpolarized capacitor"
-			(at 163.83 105.41 0)
-			(hide yes)
+		(property "Description" ""
+			(at 166.37 109.22 0)
 			(show_name no)
 			(do_not_autoplace no)
@@
 			)
 		)
-		(property "Value" "10u"
+		(property "Value" "10u 50V"
 			(at 176.53 101.6 0)
 			(show_name no)
@@
 			)
 		)
-		(property "Footprint" ""
+		(property "Footprint" "SamacSys_Parts:RDEC71H106K3K1H03B"
 			(at 176.2252 109.22 0)
 			(hide yes)
@@
 			)
 		)
-		(property "Description" "Unpolarized capacitor"
-			(at 175.26 105.41 0)
-			(hide yes)
-			(show_name no)
-			(do_not_autoplace no)
+		(property "Description" ""
+			(at 177.8 109.22 0)
+			(show_name no)
+			(do_not_autoplace no)

Commit message: version 2.0.0
Changed lines of the file:
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@@
 			)
 		)
-		(property "Description" ""
+		(property "Description" "Unpolarized capacitor"
 			(at 204.47 109.22 0)
 			(show_name no)
@@
 			)
 		)
-		(property "Description" ""
+		(property "Description" "Polarized capacitor"
 			(at 190.5 109.22 0)
 			(show_name no)
@@
 			)
 		)
-		(property "Description" ""
+		(property "Description" "Polarized capacitor"
 			(at 190.5 91.44 0)
 			(show_name no)
@@
 			)
 		)
-		(property "Description" ""
+		(property "Description" "Unpolarized capacitor"
 			(at 118.11 107.95 0)
 			(show_name no)
@@
 			)
 		)
-		(property "Description" ""
+		(property "Description" "Unpolarized capacitor"
 			(at 177.8 91.44 0)
 			(show_name no)
@@
 			)
 		)
-		(property "Description" ""
+		(property "Description" "Unpolarized capacitor"
 			(at 204.47 91.44 0)
 			(show_name no)
@@
 			)
 		)
-		(property "Description" ""
+		(property "Description" "Unpolarized capacitor"
 			(at 166.37 91.44 0)
 			(show_name no)
@@
 			)
 		)
-		(property "Description" ""
+		(property "Description" "Unpolarized capacitor"
 			(at 166.37 109.22 0)
 			(show_name no)
@@
 			)
 		)
-		(property "Description" ""
+		(property "Description" "Unpolarized capacitor"
 			(at 177.8 109.22 0)
 			(show_name no)
